Commit message: improve random_household_pick

File: helping_hands_rl_envs/simulators/urdf/object/random_household_object/boat/boat.urdf (robot description, URDF)
Before this commit: robot obj, 1 links, 0 joints
Links:
- link baseLink: geometry collision mesh filename=boat11.obj scale=0.2 0.2 0.3; visual mesh filename=boat11.obj scale=0.2 0.2 0.3

File: helping_hands_rl_envs/simulators/urdf/object/random_household_object/car/car.urdf (robot description, URDF)
Before this commit: robot obj, 1 links, 0 joints
Links:
- link baseLink: geometry collision mesh filename=car1.obj scale=0.2 0.2 0.3; visual mesh filename=car1.obj scale=0.2 0.2 0.3
