Commit message: increase kuka gripper friction, remove/add some objects in random household object set, decrease pick_offset in random_household_picking_env

File: helping_hands_rl_envs/simulators/urdf/object/random_household_object/car/car.urdf (robot description, URDF)
Before this commit: robot obj, 1 links, 0 joints
Links:
- link baseLink: geometry collision mesh filename=car4.obj scale=0.2 0.2 0.2; visual mesh filename=car4.obj scale=0.2 0.2 0.2

File: helping_hands_rl_envs/simulators/urdf/object/random_household_object/carrot/carrot.urdf (robot description, URDF)
Before this commit: robot obj, 1 links, 0 joints
Links:
- link baseLink: geometry collision mesh filename=carrot1.obj scale=0.15 0.15 0.15; visual mesh filename=carrot1.obj scale=0.15 0.15 0.15

File: helping_hands_rl_envs/simulators/urdf/object/random_household_object/cask/cask.urdf (robot description, URDF)
Before this commit: robot obj, 1 links, 0 joints
Links:
- link baseLink: geometry collision mesh filename=cask1.obj scale=0.1 0.1 0.1; visual mesh filename=cask1.obj scale=0.1 0.1 0.1

File: helping_hands_rl_envs/simulators/urdf/object/random_household_object/croissant/croissant.urdf (robot description, URDF)
Before this commit: robot obj, 1 links, 0 joints
Links:
- link baseLink: geometry collision mesh filename=croissant.obj scale=0.15 0.15 0.25; visual mesh filename=croissant.obj scale=0.15 0.15 0.25

File: helping_hands_rl_envs/simulators/urdf/object/random_household_object/donut/donut.urdf (robot description, URDF)
Before this commit: robot obj, 1 links, 0 joints
Links:
- link baseLink: geometry collision mesh filename=donut2.obj scale=0.1 0.1 0.1; visual mesh filename=donut2.obj scale=0.1 0.1 0.15

File: helping_hands_rl_envs/simulators/urdf/object/random_household_object/flashlight/flashlight.urdf (robot description, URDF)
Before this commit: robot obj, 1 links, 0 joints
Links:
- link baseLink: geometry collision mesh filename=flashlight1.obj scale=0.25 0.15 0.25; visual mesh filename=flashlight1.obj scale=0.25 0.15 0.25
