Commit message: adjusted object appearances; cylinder is now similar size as cube, to allow for stacking

File: helping_hands_rl_envs/simulators/urdf/object/cylinder.urdf (robot description, URDF)
Before this commit: robot cylinder.urdf, 1 links, 0 joints
Links:
- link baseLink: geometry collision cylinder length=0.05 radius=0.025; visual cylinder length=0.05 radius=0.025
