Commit message: box palletizing: decrease box length, increase rz restriction

File: helping_hands_rl_envs/simulators/urdf/object/box/box.urdf (robot description, URDF)
Before this commit: robot box.urdf, 1 links, 0 joints
Links:
- link baseLink: geometry collision box size=0.056 0.0875 0.056; visual box size=0.056 0.0875 0.056

Commit message: decrease box size and gap

File: helping_hands_rl_envs/simulators/urdf/object/box/box.urdf (robot description, URDF)
Before this commit: robot box.urdf, 1 links, 0 joints
Links:
- link baseLink: geometry collision box size=0.055 0.0865 0.055; visual box size=0.055 0.0865 0.055
