Commit message: Adding square peg insertion env. Testing new force physics simulation settings to reduce object penetration.

File: helping_hands_rl_envs/pybullet/urdf/object/square_peg.urdf (robot description, URDF)
Before this commit: robot peg.urdf, 1 links, 0 joints
Links:
- link baseLink: geometry collision mesh filename=cube.obj scale=0.5 0.5 1.0; visual mesh filename=cube.obj scale=0.5 0.5 1.0

Commit message: Minor updates to peg insertion env

File: helping_hands_rl_envs/pybullet/urdf/object/square_peg.urdf (robot description, URDF)
Before this commit: robot square_peg.urdf, 1 links, 0 joints
Links:
- link baseLink: geometry collision mesh filename=cube.obj scale=0.5 0.5 0.9; visual mesh filename=cube.obj scale=0.5 0.5 0.9
