Commit message: Good gripper orientation on arm

File: helping_hands_rl_envs/simulators/urdf/ur5/ur5_hydrostatic_gripper.urdf (robot description, URDF)
Before this commit: robot assembled_robot, 12 links, 11 joints
Links:
- added link dummy_center_indicator_link, mass 0.0; visual box size=0.02 0.02 0.02
- added link narrow_finger_link, mass 0.016641; collision mesh filename=simulators/urdf/hydrostatic_gripper/meshes/narrow_finger.STL; visual mesh filename=simulators/urdf/hydrostatic_gripper/meshes/narrow_finger.STL
- added link wide_finger_link, mass 0.0167; collision mesh filename=simulators/urdf/hydrostatic_gripper/meshes/wide_finger.STL; visual mesh filename=simulators/urdf/hydrostatic_gripper/meshes/wide_finger.STL
- link gripah_base: geometry collision mesh filename=simulators/urdf/hydrostatic_gripper/meshes/wrist.STL; visual mesh filename=simulators/urdf/hydrostatic_gripper/meshes/wrist.STL
Joints:
- added joint dummy_center_fixed_joint: type fixed, parent simple_arm_tool0, child dummy_center_indicator_link, origin xyz=0 -0.2 0.015 rpy=0.0 0.0 1.5707
- added joint narrow_finger_joint: type revolute, parent gripah_base, child narrow_finger_link, origin xyz=0.055 0 0 rpy=1.5708 0.013333 8.164E-19, axis 0 0 -1, limit lower=-1.0472 upper=1.0472 effort=6.6 velocity=8.0
- added joint wide_finger_joint: type revolute, parent gripah_base, child wide_finger_link, origin xyz=0.055 0 0 rpy=1.5708 0.013333 -8.164E-19, axis 0 0 1, limit lower=-1.0472 upper=1.0472 effort=6.6 velocity=8.0
- joint simple_arm_tool0_simple_gripper_base_joint: origin xyz=0 0 0 rpy=0 -1.5708 0 -> xyz=0 0 0.015 rpy=1.5708 0 -1.5708

Commit message: Gripper orientation lifelike

File: helping_hands_rl_envs/simulators/urdf/ur5/ur5_hydrostatic_gripper.urdf (robot description, URDF)
Before this commit: robot assembled_robot, 15 links, 14 joints
Joints:
- joint simple_arm_tool0_simple_gripper_base_joint: origin xyz=0 0 0.015 rpy=1.5708 0 -1.5708 -> xyz=0 0 0.015 rpy=0.785398 0 -1.5708

Commit message: Add ur5 hydristatic gripper robot class

File: helping_hands_rl_envs/simulators/urdf/ur5/ur5_hydrostatic_gripper.urdf (robot description, URDF)
Before this commit: robot assembled_robot, 15 links, 14 joints
Joints:
- joint dummy_center_fixed_joint: origin xyz=0 -0.2 0.015 rpy=0.0 0.0 1.5707 -> xyz=0 -0.2 0.015 rpy=0.785398 0.0 1.5707

Commit message: Correct grasp positioning link orientation

File: helping_hands_rl_envs/simulators/urdf/ur5/ur5_hydrostatic_gripper.urdf (robot description, URDF)
Before this commit: robot assembled_robot, 15 links, 14 joints
Joints:
- joint dummy_center_fixed_joint: origin xyz=0 -0.2 0.015 rpy=0.785398 0.0 1.5707 -> xyz=0 -0.2 0.015 rpy=-1.5707 0.785398 0.0
