Commit message: Add ur5 with new gripper

File: helping_hands_rl_envs/simulators/urdf/hydrostatic_gripper_2/urdf/hydrostatic_gripper_v2.urdf (robot description, URDF)
Before this commit: robot Gripper_v3.SLDASM, 9 links, 8 joints
Joints:
- joint dummy_ee_joint: origin xyz=0.150013332741805 0 0 rpy=0 1.5707963267949 0 -> xyz=0.14 0 0 rpy=0 1.5707963267949 0
