Commit message: Added new ur5 + gripper model.

File: helping_hands_rl_envs/pybullet/urdf/ur5/ur5_hydrostatic_gripper.urdf (robot description, URDF)
Before this commit: robot assembled_robot, 15 links, 14 joints
Links:
- removed link dummy_center_indicator_link
- removed link gripah_base
- removed link narrow_finger_link
- removed link wide_finger_link
- added link dummy_ee_link; visual box size=0.01 0.01 0.01
- added link gripper_base, mass 0.786634201066895; collision mesh filename=helping_hands_rl_envs/pybullet/urdf/hydrostatic_gripper/mes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; visual mesh filename=helping_hands_rl_envs/pybullet/urdf/hydrostatic_gripper/mes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
- added link gripper_wrist_addapter, mass 0.0139506047612529; collision mesh filename=helping_hands_rl_envs/pybullet/urdf/hydrostatic_gripper/mes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; visual mesh filename=helping_hands_rl_envs/pybullet/urdf/hydrostatic_gripper/mes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
- added link left_finger_base, mass 0.0110794759852593; collision mesh filename=helping_hands_rl_envs/pybullet/urdf/hydrostatic_gripper/mes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; visual mesh filename=helping_hands_rl_envs/pybullet/urdf/hydrostatic_gripper/mes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
- added link left_finger_mid, mass 0.00233205195898081; collision mesh filename=helping_hands_rl_envs/pybullet/urdf/hydrostatic_gripper/mes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; visual mesh filename=helping_hands_rl_envs/pybullet/urdf/hydrostatic_gripper/mes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
- added link left_finger_tip, mass 0.0032882898385146; collision mesh filename=helping_hands_rl_envs/pybullet/urdf/hydrostatic_gripper/mes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; visual mesh filename=helping_hands_rl_envs/pybullet/urdf/hydrostatic_gripper/mes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
- added link right_finger_base, mass 0.0110794759852594; collision mesh filename=helping_hands_rl_envs/pybullet/urdf/hydrostatic_gripper/mes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; visual mesh filename=helping_hands_rl_envs/pybullet/urdf/hydrostatic_gripper/mes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
- added link right_finger_mid, mass 0.00233205195898081; collision mesh filename=helping_hands_rl_envs/pybullet/urdf/hydrostatic_gripper/mes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; visual mesh filename=helping_hands_rl_envs/pybullet/urdf/hydrostatic_gripper/mes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
- added link right_finger_tip, mass 0.0032882898385146; collision mesh filename=helping_hands_rl_envs/pybullet/urdf/hydrostatic_gripper/mes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; visual mesh filename=helping_hands_rl_envs/pybullet/urdf/hydrostatic_gripper/mes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
Joints:
- removed joint dummy_center_fixed_joint
- removed joint narrow_finger_joint
- removed joint wide_finger_joint
- added joint dummy_ee_joint: type fixed, parent gripper_base, child dummy_ee_link, origin xyz=0.150013332741805 0 0 rpy=0 1.5707963267949 0, axis 0 0 0
- added joint gripper_wrist_to_base: type fixed, parent gripper_wrist_addapter, child gripper_base, origin xyz=0.055 -0.0332705627484773 -0.016970562748477 rpy=2.35619449019234 0 0, axis 0 0 0
- added joint left_finger_base_to_mid: type fixed, parent left_finger_base, child left_finger_mid, origin xyz=0 0 0 rpy=0 0 0, axis 0 0 0
- added joint left_finger_joint: type revolute, parent gripper_base, child left_finger_base, origin xyz=0 0 0 rpy=-3.1416 0 0.013333, axis 0 0 1, limit lower=-2 upper=2 effort=0 velocity=0
- added joint left_finger_mid_to_tip: type fixed, parent left_finger_mid, child left_finger_tip, origin xyz=0 0 0 rpy=0 0 0, axis 0 0 0
- added joint right_finger_base_to_mid: type fixed, parent right_finger_base, child right_finger_mid, origin xyz=0 0 0 rpy=0 0 0, axis 0 0 0
- added joint right_finger_joint: type revolute, parent gripper_base, child right_finger_base, origin xyz=0 0 0 rpy=0 0 -0.013333, axis 0 0 -1, limit lower=-2 upper=2 effort=0 velocity=0
- added joint right_finger_mid_to_tip: type fixed, parent right_finger_mid, child right_finger_tip, origin xyz=0 0 0 rpy=0 0 0, axis 0 0 0
- joint simple_arm_tool0_simple_gripper_base_joint: child gripah_base -> gripper_wrist_addapter; origin xyz=0 0 0.015 rpy=0.785398 0 -1.5708 -> xyz=0 0 0 rpy=-1.570796 0 3.141593

Commit message: invert gripper joint axis to make more intiitive sense

File: helping_hands_rl_envs/pybullet/urdf/ur5/ur5_hydrostatic_gripper.urdf (robot description, URDF)
Before this commit: robot assembled_robot, 20 links, 19 joints
Joints:
- joint right_finger_joint: axis 0 0 -1 -> 0 0 1

Commit message: Invert gripper ee link frame

File: helping_hands_rl_envs/pybullet/urdf/ur5/ur5_hydrostatic_gripper.urdf (robot description, URDF)
Before this commit: robot assembled_robot, 20 links, 19 joints
Joints:
- joint dummy_ee_joint: origin xyz=0.150013332741805 0 0 rpy=0 1.5707963267949 0 -> xyz=0.150013332741805 0 0 rpy=3.141593 1.5707963267949 0

Commit message: Force updates

File: helping_hands_rl_envs/pybullet/urdf/ur5/ur5_hydrostatic_gripper.urdf (robot description, URDF)
Before this commit: robot assembled_robot, 20 links, 19 joints
Links:
- link dummy_ee_link: geometry 

Commit message: Fixed rotation of gripper finger img in ur5 w/hydrostatic gripper. Started refactoring robots a bit.

File: helping_hands_rl_envs/pybullet/urdf/ur5/ur5_hydrostatic_gripper.urdf (robot description, URDF)
Before this commit: robot assembled_robot, 20 links, 19 joints
Joints:
- joint dummy_ee_joint: axis 0 0 0 -> (none)
