Commit message: Trying to fix bug where panda does not have force senseing along gripper closing joint

File: helping_hands_rl_envs/pybullet/urdf/franka_panda/panda.urdf (robot description, URDF)
Before this commit: robot panda, 13 links, 12 joints
Links:
- added link panda_left_finger, mass 0.1
- added link panda_right_finger, mass 0.1
Joints:
- added joint panda_left_finger: type fixed, parent panda_leftfinger, child panda_left_finger, origin xyz=0 0 0 rpy=0 0 0
- added joint panda_right_finger: type fixed, parent panda_rightfinger, child panda_right_finger, origin xyz=0 0 0 rpy=0 0 0

Commit message: Testing force map reprentation

File: helping_hands_rl_envs/pybullet/urdf/franka_panda/panda.urdf (robot description, URDF)
Before this commit: robot panda, 15 links, 14 joints
Links:
- link panda_left_finger: geometry visual box size=0.01 0.01 0.01
- link panda_right_finger: geometry visual box size=0.01 0.01 0.01
Joints:
- joint panda_left_finger: origin xyz=0 0 0 rpy=0 0 0 -> xyz=0 0 0.0584 rpy=0 0 0; parent panda_leftfinger -> panda_hand
- joint panda_right_finger: origin xyz=0 0 0 rpy=0 0 0 -> xyz=0 0 0.0584 rpy=0 0 0; parent panda_rightfinger -> panda_hand

Commit message: Trying to fix finger joint force sensing

File: helping_hands_rl_envs/pybullet/urdf/franka_panda/panda.urdf (robot description, URDF)
Before this commit: robot panda, 15 links, 14 joints
Links:
- link panda_left_finger: geometry visual box size=0.00 0.00 0.00
- link panda_right_finger: geometry visual box size=0.0 0.0 0.0
Joints:
- joint panda_finger_joint1: parent panda_hand -> panda_left_finger
- joint panda_finger_joint2: parent panda_hand -> panda_right_finger
- joint panda_left_finger: origin xyz=0 0 0.0584 rpy=0 0 0 -> xyz=0 0.0 0.0 rpy=0 0 0
- joint panda_right_finger: origin xyz=0 0 0.0584 rpy=0 0 0 -> xyz=0 0.0 0.0 rpy=0 0 0

Commit message: New force test chages for block pulling.

File: helping_hands_rl_envs/pybullet/urdf/franka_panda/panda.urdf (robot description, URDF)
Before this commit: robot panda, 15 links, 14 joints
Joints:
- joint panda_grasptarget_hand: origin xyz=0 0 0.105 rpy=3.1415 0 1.5707 -> xyz=0 0 0.105 rpy=3.1415 0 1.675

Commit message: Trying to mask out panda gripper better.

File: helping_hands_rl_envs/pybullet/urdf/franka_panda/panda.urdf (robot description, URDF)
Before this commit: robot panda, 15 links, 14 joints
Links:
- link panda_leftfinger: geometry collision mesh filename=package://meshes/collision/finger.obj
- link panda_rightfinger: geometry collision mesh filename=package://meshes/collision/finger.obj
Joints:
- joint panda_grasptarget_hand: origin xyz=0 0 0.105 rpy=3.1415 0 1.675 -> xyz=0 0 0.105 rpy=3.1415 0 1.5707

Commit message: Hiding panda finger for the moment as masking them out is just miserable

File: helping_hands_rl_envs/pybullet/urdf/franka_panda/panda.urdf (robot description, URDF)
Before this commit: robot panda, 15 links, 14 joints
Links:
- link panda_leftfinger: geometry collision mesh filename=package://meshes/collision/finger.obj; visual box size=0.00 0.00 0.00
- link panda_rightfinger: geometry collision mesh filename=package://meshes/collision/finger.obj; visual box size=0.00 0.00 0.00

Commit message: Removing more visual aspects from panda due to masking issues

File: helping_hands_rl_envs/pybullet/urdf/franka_panda/panda.urdf (robot description, URDF)
Before this commit: robot panda, 15 links, 14 joints
Links:
- link panda_hand: geometry collision mesh filename=package://meshes/collision/hand.obj; visual box size=0.00 0.00 0.00
